Commit message: added robotstatepubblisher with more files in another package and found outy the front wheels not moving error but couldn't solve it

File: Files/01-myfirst.urdf (robot description, URDF)
Before this commit: robot Bobby, 7 links, 6 joints
Links:
- removed link front_wheel
- added link front_left_wheel, mass 1; collision cylinder length=0.05 radius=0.035; visual cylinder length=0.05 radius=0.035
- added link front_right_wheel, mass 1; collision cylinder length=0.05 radius=0.035; visual cylinder length=0.05 radius=0.035
- link center_thing: mass 5 -> 0.5
- link left_thing: mass 5 -> 0.5
- link right_thing: mass 5 -> 0.5
Joints:
- removed joint front_wheel_joint
- added joint front_left_wheel_joint: type continuous, parent base_link, child front_left_wheel, origin xyz=0.1 -0.15 -0.085 rpy=0 0 0, axis 0 1 0
- added joint front_right_wheel_joint: type continuous, parent base_link, child front_right_wheel, origin xyz=0.1 0.15 -0.085 rpy=0 0 0, axis 0 1 0

Commit message: changed the inertial values again and mass for base but still same problem as before

File: Files/01-myfirst.urdf (robot description, URDF)
Before this commit: robot Bobby, 8 links, 7 joints
Links:
- link base_link: mass 20 -> 10
- link center_thing: mass 0.5 -> 0.1
- link left_thing: mass 0.5 -> 0.1
- link right_thing: mass 0.5 -> 0.1
